Commit message: add colors to robot model

File: my_robot/urdf/my_robot.xacro (robot description, xacro)
@@ -30,4 +30,7 @@
         <box size=".4 .2 .1"/>
       </geometry>
+      <material name="blue">
+          <color rgba="0.0 0.0 1.0 1.0"/>
+      </material>
     </visual>
     <collision name='back_caster_collision'>
@@ -76,4 +79,7 @@
         <cylinder radius="0.1" length="0.05"/>
       </geometry>
+      <material name="green">
+        <color rgba="0 1.0 0 1.0"/>
+      </material>
     </visual>
   </link>
@@ -98,4 +104,7 @@
         <cylinder radius="0.1" length="0.05"/>
       </geometry>
+      <material name="green">
+        <color rgba="0 1.0 0 1.0"/>
+      </material>
     </visual>
   </link>
@@ -120,4 +129,7 @@
         <box size="0.05 0.05 0.05" />
       </geometry>
+      <material name="red">
+        <color rgba="1.0 0 0 1.0"/>
+      </material>
     </visual>
   </link>

Commit message: edit robot model to differ from lesson's one

File: my_robot/urdf/my_robot.xacro (robot description, xacro)
@@ -22,5 +22,6 @@
       <origin xyz="0 0 0" rpy=" 0 0 0"/>
       <geometry>
-        <box size=".4 .2 .1"/>
+        <!--<box size=".4 .2 .1"/>-->
+        <cylinder radius="0.15" length="0.1"/>
       </geometry>
     </collision>
@@ -28,12 +29,14 @@
       <origin xyz="0 0 0" rpy=" 0 0 0"/>
       <geometry>
-        <box size=".4 .2 .1"/>
+        <!--<box size=".4 .2 .1"/>-->
+        <cylinder radius="0.15" length="0.2"/>
       </geometry>
-      <material name="blue">
-          <color rgba="0.0 0.0 1.0 1.0"/>
+      <material name="red">
+          <color rgba="1.0 0.0 0.0 1.0"/>
       </material>
     </visual>
     <collision name='back_caster_collision'>
-      <origin xyz="-0.15 0 -0.05" rpy=" 0 0 0"/>
+      <!-- <origin xyz="-0.15 0 -0.05" rpy=" 0 0 0"/> -->
+      <origin xyz="-0.08 0 -0.05" rpy=" 0 0 0"/>
       <geometry>
         <sphere radius="0.0499"/>
@@ -41,5 +44,6 @@
     </collision>
     <visual name='back_caster_visual'>
-      <origin xyz="-0.15 0 -0.05" rpy=" 0 0 0"/>
+      <!-- <origin xyz="-0.15 0 -0.05" rpy=" 0 0 0"/> -->
+      <origin xyz="-0.08 0 -0.05" rpy=" 0 0 0"/>
       <geometry>
         <sphere radius="0.05"/>
@@ -47,5 +51,6 @@
     </visual>
     <collision name='front_caster_collision'>
-      <origin xyz="0.15 0 -0.05" rpy=" 0 0 0"/>
+      <!-- <origin xyz="0.15 0 -0.05" rpy=" 0 0 0"/> -->
+      <origin xyz="0.08 0 -0.05" rpy=" 0 0 0"/>
       <geometry>
         <sphere radius="0.0499"/>
@@ -53,5 +58,6 @@
     </collision>
     <visual name='front_caster_visual'>
-      <origin xyz="0.15 0 -0.05" rpy=" 0 0 0"/>
+      <!-- <origin xyz="0.15 0 -0.05" rpy=" 0 0 0"/> -->
+      <origin xyz="0.08 0 -0.05" rpy=" 0 0 0"/>
       <geometry>
         <sphere radius="0.05"/>
@@ -129,6 +135,6 @@
         <box size="0.05 0.05 0.05" />
       </geometry>
-      <material name="red">
-        <color rgba="1.0 0 0 1.0"/>
+      <material name="blue">
+        <color rgba="0.0 0 1.0 1.0"/>
       </material>
     </visual>
@@ -158,5 +164,6 @@
   <!--Joints-->
   <joint type="continuous" name="right_wheel_hinge">
-    <origin xyz="0 0.15 0" rpy="0 0 0"/>
+    <!--<origin xyz="0 0.15 0" rpy="0 0 0"/>-->
+    <origin xyz="0 0.175 0" rpy="0 0 0"/>
     <child link="right_wheel"/>
     <parent link="chassis"/>
@@ -166,5 +173,6 @@
   </joint>
   <joint type="continuous" name="left_wheel_hinge">
-    <origin xyz="0 -0.15 0" rpy="0 0 0"/>
+    <!--<origin xyz="0 -0.15 0" rpy="0 0 0"/>-->
+    <origin xyz="0 -0.175 0" rpy="0 0 0"/>
     <child link="left_wheel"/>
     <parent link="chassis"/>
@@ -174,5 +182,6 @@
   </joint>
   <joint type="fixed" name="camera_joint">
-    <origin xyz="0.2 0 0" rpy="0 0 0" />
+    <!--<origin xyz="0.2 0 0" rpy="0 0 0" />-->
+    <origin xyz="0.15 0 0" rpy="0 0 0" />
     <child link="camera" />
     <parent link="chassis" />
@@ -180,5 +189,6 @@
   </joint>
   <joint type="fixed" name="hokuyo_joint">
-    <origin xyz="0.15 0 0.1" rpy="0 0 0" />
+    <!--<origin xyz="0.15 0 0.1" rpy="0 0 0" />-->
+    <origin xyz="0.08 0 0.15" rpy="0 0 0" />
     <child link="hokuyo" />
     <parent link="chassis" />

Commit message: chenge robot model to be more stable

File: my_robot/urdf/my_robot.xacro (robot description, xacro)
@@ -22,5 +22,4 @@
       <origin xyz="0 0 0" rpy=" 0 0 0"/>
       <geometry>
-        <!--<box size=".4 .2 .1"/>-->
         <cylinder radius="0.15" length="0.1"/>
       </geometry>
@@ -29,6 +28,5 @@
       <origin xyz="0 0 0" rpy=" 0 0 0"/>
       <geometry>
-        <!--<box size=".4 .2 .1"/>-->
-        <cylinder radius="0.15" length="0.2"/>
+        <cylinder radius="0.15" length="0.1"/>
       </geometry>
       <material name="red">
@@ -37,6 +35,5 @@
     </visual>
     <collision name='back_caster_collision'>
-      <!-- <origin xyz="-0.15 0 -0.05" rpy=" 0 0 0"/> -->
-      <origin xyz="-0.08 0 -0.05" rpy=" 0 0 0"/>
+      <origin xyz="-0.095 0 -0.05" rpy=" 0 0 0"/>
       <geometry>
         <sphere radius="0.0499"/>
@@ -44,6 +41,5 @@
     </collision>
     <visual name='back_caster_visual'>
-      <!-- <origin xyz="-0.15 0 -0.05" rpy=" 0 0 0"/> -->
-      <origin xyz="-0.08 0 -0.05" rpy=" 0 0 0"/>
+      <origin xyz="-0.095 0 -0.05" rpy=" 0 0 0"/>
       <geometry>
         <sphere radius="0.05"/>
@@ -51,6 +47,5 @@
     </visual>
     <collision name='front_caster_collision'>
-      <!-- <origin xyz="0.15 0 -0.05" rpy=" 0 0 0"/> -->
-      <origin xyz="0.08 0 -0.05" rpy=" 0 0 0"/>
+      <origin xyz="0.095 0 -0.05" rpy=" 0 0 0"/>
       <geometry>
         <sphere radius="0.0499"/>
@@ -58,6 +53,5 @@
     </collision>
     <visual name='front_caster_visual'>
-      <!-- <origin xyz="0.15 0 -0.05" rpy=" 0 0 0"/> -->
-      <origin xyz="0.08 0 -0.05" rpy=" 0 0 0"/>
+      <origin xyz="0.095 0 -0.05" rpy=" 0 0 0"/>
       <geometry>
         <sphere radius="0.05"/>
@@ -164,6 +158,5 @@
   <!--Joints-->
   <joint type="continuous" name="right_wheel_hinge">
-    <!--<origin xyz="0 0.15 0" rpy="0 0 0"/>-->
-    <origin xyz="0 0.175 0" rpy="0 0 0"/>
+    <origin xyz="0 0.15 0" rpy="0 0 0"/>
     <child link="right_wheel"/>
     <parent link="chassis"/>
@@ -173,6 +166,5 @@
   </joint>
   <joint type="continuous" name="left_wheel_hinge">
-    <!--<origin xyz="0 -0.15 0" rpy="0 0 0"/>-->
-    <origin xyz="0 -0.175 0" rpy="0 0 0"/>
+    <origin xyz="0 -0.15 0" rpy="0 0 0"/>
     <child link="left_wheel"/>
     <parent link="chassis"/>
@@ -182,5 +174,4 @@
   </joint>
   <joint type="fixed" name="camera_joint">
-    <!--<origin xyz="0.2 0 0" rpy="0 0 0" />-->
     <origin xyz="0.15 0 0" rpy="0 0 0" />
     <child link="camera" />
@@ -189,6 +180,5 @@
   </joint>
   <joint type="fixed" name="hokuyo_joint">
-    <!--<origin xyz="0.15 0 0.1" rpy="0 0 0" />-->
-    <origin xyz="0.08 0 0.15" rpy="0 0 0" />
+    <origin xyz="0.08 0 0.1" rpy="0 0 0" />
     <child link="hokuyo" />
     <parent link="chassis" />
